File: hardware/6809ROMRAM/6809ROMRAM.kicad_pcb (KiCad board)
At the start: 2 copper layers, 100 x 100 mm, 22 parts, among them J1 SS50-LIKE, J2 Address Select, U1 628128, U2 28C256, U3 28C256, U4 628128, U5 74HC85, U6 74HC04, U7 74HC08, U8 74HC00

Commit message: ROMRAM board
Parts:
- added H1: MountingHole, MountingHole:MountingHole_3.2mm_M3_ISO14580_Pad, F.Cu at (167.6, 59.7)
- added H2: MountingHole, MountingHole:MountingHole_3.2mm_M3_ISO14580_Pad, F.Cu at (256.5, 59.7)
- added H3: MountingHole, MountingHole:MountingHole_3.2mm_M3_ISO14580_Pad, F.Cu at (167.6, 149.9)
- added H4: MountingHole, MountingHole:MountingHole_3.2mm_M3_ISO14580_Pad, F.Cu at (256.5, 149.9)
- added Logo1: Pinnated, Pinnated:Pinnule, F.Cu at (238.8, 146.1)
- moved R1 70.0 mm to (256.5, 128.3)
- moved R4 69.3 mm to (256.5, 139.7)
- moved J2 67.3 mm to (234.9, 129.5)
- moved R3 53.6 mm to (256.5, 135.9)
- moved R2 53.3 mm to (256.5, 132.1)
- moved C5 15.5 mm to (223.5, 115.6)
- moved U5 14.0 mm to (221.0, 120.7)
- moved U8 11.5 mm to (208.3, 120.7)
- moved C1 10.9 mm to (196.8, 63.5)
- moved C8 10.5 mm to (210.8, 115.6)
- moved C4 6.35 mm to (212.1, 63.5)
- moved C2 6.35 mm to (232.4, 68.6)
- moved C3 6.35 mm to (252.7, 68.6)
- moved C6 3.59 mm to (198.1, 115.6)
- moved C7 3.59 mm to (185.4, 115.6)
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Connections:
- C2 pad 1: +5v -> GND
- C2 pad 2: GND -> +5v
- C3 pad 1: +5v -> GND
- C3 pad 2: GND -> +5v
- C4 pad 1: +5v -> GND
- C4 pad 2: GND -> +5v
- C5 pad 1: +5v -> GND
- C5 pad 2: GND -> +5v
- C6 pad 1: +5v -> GND
- C6 pad 2: GND -> +5v
- C7 pad 1: +5v -> GND
- C7 pad 2: GND -> +5v
- C8 pad 1: +5v -> GND
- C8 pad 2: GND -> +5v
Routing:
- net GND: track 0.00 -> 613.8 mm
- net +5v: track 0.00 -> 371.2 mm
- net /A15: track 0.00 -> 139.0 mm, vias 0 -> 1
- net /D4: track 0.00 -> 134.2 mm, vias 0 -> 2
- net BOARD-SELECT: track 0.00 -> 132.8 mm, vias 0 -> 1
- net /D3: track 0.00 -> 132.4 mm, vias 0 -> 2
- net /D6: track 0.00 -> 129.6 mm, vias 0 -> 2
- net /D2: track 0.00 -> 129.6 mm, vias 0 -> 2
- net /D5: track 0.00 -> 128.8 mm, vias 0 -> 2
- net /D7: track 0.00 -> 124.2 mm, vias 0 -> 2
- net /D1: track 0.00 -> 119.9 mm, vias 0 -> 1
- net ~W: track 0.00 -> 119.6 mm, vias 0 -> 3
- net /D0: track 0.00 -> 117.5 mm
- net ~R: track 0.00 -> 106.9 mm, vias 0 -> 1
- net ~RAM-SELECT: track 0.00 -> 96.4 mm, vias 0 -> 1
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Other:
- board text added: "1"
- board text added: "128KB RAM | 64KB ROM/RAM Prototype 1 25 April 2021"
- board text added: "Copyrigh (c) 2021 andrew@pinnated.com"
- board text added: "Top bits of physical address 0000 Taken by sysrem, try 0001 Jumper in place = 1"

Commit message: ground layers
Routing:
- net +5v: track 371.2 -> 369.9 mm
- added copper zone on B.Cu, net GND
- added copper zone on F.Cu, net GND
Other:
- board text added: "A17"
- board text added: "A18"
- board text added: "A19"
- board text added: "A20"
- board text added: "RAM 2 & 3"
- board text added: "RAM only"
- board text added: "ROM 0"
- board text added: "ROM 1"
- board text added: "Top bits of physical address 0000 Taken by system Start at 0001 Jumper = 1, No jumper = 0 Order in memory: 32K ROM 0, 32K ROM 1, 64K RAM"
- board text removed: "Top bits of physical address 0000 Taken by sysrem, try 0001 Jumper in place = 1"
Changed lines of the file:
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@@
   (general
     (thickness 1.6)
-    (drawings 8)
-    (tracks 945)
+    (drawings 17)
+    (tracks 944)
     (zones 0)
     (modules 27)
@@
     (47 F.CrtYd user)
     (48 B.Fab user)
-    (49 F.Fab user hide)
+    (49 F.Fab user)
   )
   (setup
@@
     )
   )
-  (gr_text "Top bits of physical address\n0000 Taken by sysrem, try 0001\nJumper in place = 1" (at 245.11 121.92) (layer F.SilkS)
+  (gr_text 1 (at 166.37 68.58) (layer F.SilkS)
+    (effects (font (size 1 1) (thickness 0.15)))
+  )
+  (gr_text A17 (at 240.931501 137.16) (layer F.SilkS)
+    (effects (font (size 1 1) (thickness 0.15)))
+  )
+  (gr_text A18 (at 240.931581 134.62) (layer F.SilkS)
+    (effects (font (size 1 1) (thickness 0.15)))
+  )
+  (gr_text A19 (at 240.931724 132.08) (layer F.SilkS)
+    (effects (font (size 1 1) (thickness 0.15)))
+  )
+  (gr_text A20 (at 240.934725 129.54) (layer F.SilkS)
+    (effects (font (size 1 1) (thickness 0.15)))
+  )
+  (gr_text "RAM 2 & 3" (at 207.01 63.5) (layer F.SilkS)
+    (effects (font (size 1 1) (thickness 0.15)))
+  )
+  (gr_text "ROM 1" (at 243.84 69.85) (layer F.SilkS)
+    (effects (font (size 1 1) (thickness 0.15)))
+  )
+  (gr_text "ROM 0" (at 223.52 69.85) (layer F.SilkS)
+    (effects (font (size 1 1) (thickness 0.15)))
+  )
+  (gr_text "RAM only" (at 189.23 63.5) (layer F.SilkS)
+    (effects (font (size 1 1) (thickness 0.15)))
+  )
+  (gr_text "Top bits of physical address\n0000 Taken by system\nStart at 0001\nJumper = 1, No jumper = 0\nOrder in memory:\n32K ROM 0, 32K ROM 1, 64K RAM" (at 243.84 120.65) (layer F.SilkS)
     (effects (font (size 1 1) (thickness 0.15)))
   )
@@
   (segment (start 251.46 66.04) (end 255.27 66.04) (width 1) (layer B.Cu) (net 22))
   (segment (start 257.81 68.58) (end 257.81 73.66) (width 1) (layer B.Cu) (net 22))
-  (segment (start 257.81 73.66) (end 256.54 73.66) (width 0.25) (layer B.Cu) (net 22))
   (segment (start 234.95 129.54) (end 234.95 132.08) (width 1) (layer F.Cu) (net 22))
   (segment (start 234.95 132.08) (end 234.95 134.62) (width 1) (layer F.Cu) (net 22))
   (segment (start 234.95 134.62) (end 234.95 137.16) (width 1) (layer F.Cu) (net 22))
-  (segment (start 257.81 73.66) (end 259.08 73.66) (width 0.25) (layer F.Cu) (net 22))
+  (segment (start 257.81 73.66) (end 259.08 73.66) (width 1) (layer F.Cu) (net 22))
   (segment (start 259.08 73.66) (end 260.35 74.93) (width 1) (layer F.Cu) (net 22))
   (segment (start 228.6 115.49) (end 228.52 115.57) (width 0.25) (layer F.Cu) (net 22))
@@
   (segment (start 214.63 72.39) (end 201.93 72.39) (width 0.25) (layer F.Cu) (net 42))
   (segment (start 215.9 71.12) (end 217.17 71.12) (width 0.25) (layer F.Cu) (net 42))
-  (segment (start 205.74 120.65) (end 208.28 123.19) (width 0.25) (layer B.Cu) (net 42))
-  (segment (start 205.74 119.38) (end 205.74 120.65) (width 0.25) (layer B.Cu) (net 42))
-  (segment (start 207.01 118.11) (end 205.74 119.38) (width 0.25) (layer B.Cu) (net 42))
   (segment (start 217.17 71.12) (end 218.44 71.12) (width 0.25) (layer B.Cu) (net 42))
   (segment (start 218.44 71.12) (end 219.71 72.39) (width 0.25) (layer B.Cu) (net 42))
   (segment (start 196.85 130.81) (end 195.58 130.81) (width 0.25) (layer B.Cu) (net 42))
   (segment (start 198.12 129.54) (end 196.85 130.81) (width 0.25) (layer B.Cu) (net 42))
-  (segment (start 205.74 124.46) (end 205.74 128.27) (width 0.25) (layer B.Cu) (net 42))
   (segment (start 204.47 129.54) (end 198.12 129.54) (width 0.25) (layer B.Cu) (net 42))
   (segment (start 205.74 128.27) (end 204.47 129.54) (width 0.25) (layer B.Cu) (net 42))
-  (segment (start 207.01 123.19) (end 205.74 124.46) (width 0.25) (layer B.Cu) (net 42))
-  (segment (start 208.28 123.19) (end 207.01 123.19) (width 0.25) (layer B.Cu) (net 42))
   (segment (start 219.71 72.39) (end 219.71 115.57) (width 0.25) (layer B.Cu) (net 42))
   (segment (start 217.17 118.11) (end 219.71 115.57) (width 0.25) (layer B.Cu) (net 42))
   (segment (start 217.17 118.11) (end 207.01 118.11) (width 0.25) (layer B.Cu) (net 42))
+  (segment (start 207.01 118.11) (end 205.74 119.38) (width 0.25) (layer B.Cu) (net 42))
+  (segment (start 205.74 119.38) (end 205.74 120.65) (width 0.25) (layer B.Cu) (net 42))
+  (segment (start 205.74 120.65) (end 208.28 123.19) (width 0.25) (layer B.Cu) (net 42))
+  (segment (start 205.74 124.46) (end 205.74 128.27) (width 0.25) (layer B.Cu) (net 42))
+  (segment (start 207.01 123.19) (end 205.74 124.46) (width 0.25) (layer B.Cu) (net 42))
+  (segment (start 208.28 123.19) (end 207.01 123.19) (width 0.25) (layer B.Cu) (net 42))
   (segment (start 195.58 96.52) (end 196.85 96.52) (width 0.25) (layer B.Cu) (net 43))
   (segment (start 194.31 95.25) (end 195.58 96.52) (width 0.25) (layer B.Cu) (net 43))
@@
   (segment (start 207.01 128.27) (end 208.28 128.27) (width 0.25) (layer F.Cu) (net 71))
   (segment (start 205.74 127) (end 207.01 128.27) (width 0.25) (layer F.Cu) (net 71))
+  (zone (net 23) (net_name GND) (layer B.Cu) (hatch edge 0.508)
+    (connect_pads (clearance 0.508))
+    (min_thickness 0.254)
+    (fill yes (arc_segments 32) (thermal_gap 0.508) (thermal_bridge_width 0.508))
+    (polygon
+      (pts
+        (xy 260.35 152.4) (xy 163.83 152.4) (xy 163.83 55.88) (xy 260.35 55.88)
+      )
+    )
+  )
+  (zone (net 23) (net_name GND) (layer F.Cu) (hatch edge 0.508)
+    (connect_pads (clearance 0.508))
+    (min_thickness 0.254)
+    (fill yes (arc_segments 32) (thermal_gap 0.508) (thermal_bridge_width 0.508))
+    (polygon
+      (pts
+        (xy 260.35 152.4) (xy 163.83 152.4) (xy 163.83 55.88) (xy 260.35 55.88)
+      )
+    )
+  )
 )
