File: hardware/6809display/6809display.kicad_pcb (KiCad board)
At the start: 2 copper layers, 99.1 x 99.1 mm, 44 parts, among them J1 Video Out, J2 To Computer, Q1 BC557, Q2 BC557, Q3 BC557, U1 74HC04, U10 74HC283, U2 74HC04, U3 74HC393, U4 SAA5020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

Commit message: clock and more
Parts:
- removed NT1: Net-Tie_2, NetTie:NetTie-2_SMD_Pad0.5mm
- R16, R17: footprint Resistor_THT:R_Axial_DIN0309_L9.0mm_D3.2mm_P12.70mm_Horizontal -> Resistor_THT:R_Axial_DIN0207_L6.3mm_D2.5mm_P7.62mm_Horizontal
- moved R17 190.8 mm to (247.7, 86.4), turned to 270 degrees
- moved R16 168.1 mm to (242.6, 86.4), turned to 270 degrees
- moved J1 127.2 mm to (271.8, 31.8), turned to 0 degrees
- moved U4 29.2 mm to (257.8, 61.0)
- moved C4 28.0 mm to (257.8, 92.7)
- moved C2 26.7 mm to (268.6, 99.1)
- moved U2 26.7 mm to (266.1, 105.4)
- moved Y1 16.6 mm to (242.6, 82.5), turned to 0 degrees
- moved C5 1.27 mm to (227.3, 55.9)
Connections:
- R17 pad 1: Net-(R16-Pad2) -> Net-(R17-Pad1)
- R17 pad 2: Net-(R17-Pad2) -> Net-(R16-Pad2)
- U1 pad 4: Net-(R17-Pad2) -> Net-(R17-Pad1)
- U4 pad 2: Net-(R17-Pad2) -> Net-(R17-Pad1)
- U5 pad 2: Net-(NT1-Pad2) -> GND
- Y1 pad 2: Net-(R17-Pad2) -> Net-(R17-Pad1)
Routing:
- net GND: track 229.1 -> 390.3 mm, vias 1 -> 3
- net +5v: track 152.6 -> 296.5 mm
- net /SA2: track 13.0 -> 135.0 mm, vias 2 -> 4
- net /SA4: track 36.5 -> 157.8 mm, vias 1 -> 5
- net /SA3: track 19.9 -> 137.3 mm, vias 0 -> 3
- net /SA1: track 6.35 -> 103.9 mm, vias 0 -> 2
- net /CA11: track 0.00 -> 95.2 mm, vias 0 -> 2
- net Net-(U1-Pad9): track 0.00 -> 81.9 mm, vias 0 -> 3
- net Net-(U1-Pad5): track 0.00 -> 80.0 mm, vias 0 -> 2
- net /A0: track 0.00 -> 71.7 mm, vias 0 -> 1
- net Net-(U4-Pad15): track 0.00 -> 70.4 mm, vias 0 -> 2
- net /A2: track 0.00 -> 70.0 mm, vias 0 -> 2
- net Net-(U4-Pad14): track 0.00 -> 69.1 mm, vias 0 -> 3
- net Net-(R17-Pad1): track 0.00 -> 69.0 mm, vias 0 -> 3
- net /A1: track 0.00 -> 68.2 mm, vias 0 -> 1
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
Commit message: digital logic wired up
Parts:
- R1, R10, R11, R12, R13, R14, R15, R2, R3, R4, R5, R6, R7, R8, R9: footprint Resistor_THT:R_Axial_DIN0309_L9.0mm_D3.2mm_P12.70mm_Horizontal -> Resistor_THT:R_Axial_DIN0207_L6.3mm_D2.5mm_P7.62mm_Horizontal
- moved R1 358.7 mm to (417.3, 29.9)
- moved R7 358.7 mm to (401.4, 30.2)
- moved Q3 305.3 mm to (353.1, 63.5)
- moved Q2 286.4 mm to (346.7, 61.0)
- moved R15 274.5 mm to (343.4, -0.59)
- moved R8 274.5 mm to (343.4, 4.16)
- moved R11 274.5 mm to (344.2, 8.91)
- moved R13 274.5 mm to (344.2, 13.7)
- moved R2 272.8 mm to (390.9, -6.00)
- moved R4 272.8 mm to (390.9, -1.25)
- moved R5 272.8 mm to (390.9, 3.50)
- moved R6 272.8 mm to (390.9, 8.25)
- moved R10 272.1 mm to (376.8, 2.91)
- moved R14 272.1 mm to (376.8, 7.66)
- moved R9 272.1 mm to (376.8, -1.84)
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Routing:
- net GND: track 390.3 -> 520.4 mm, vias 3 -> 7
- net Net-(U1-Pad12): track 0.00 -> 122.3 mm, vias 0 -> 4
- net ~Slot-Select: track 0.00 -> 120.2 mm, vias 0 -> 3
- net +5v: track 296.5 -> 339.0 mm, vias 0 -> 4
- net Net-(U10-Pad3): track 45.6 -> 61.9 mm, vias 1 -> 2
- net Net-(R17-Pad1): track 69.0 -> 64.3 mm, vias 3 -> 4
- net /CA11: track 95.2 -> 99.7 mm, vias 2 -> 4
- net /A2: track 70.0 -> 73.8 mm
- net Net-(U4-Pad13): track 55.8 -> 52.7 mm, vias 1 -> 0
- net /A0: track 71.7 -> 68.9 mm
- net Net-(U4-Pad14): track 69.1 -> 66.6 mm
- net /SA3: track 137.3 -> 134.8 mm
- net /SA4: track 157.8 -> 155.4 mm, vias 5 -> 3
- net /SA1: track 103.9 -> 101.7 mm
- net /CA4: track 26.8 -> 24.5 mm
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
Commit message: has a placement overlap
Parts:
- moved R1 179.8 mm to (237.5, 30.5), turned to 270 degrees
- moved R6 156.8 mm to (237.5, 40.6), turned to 270 degrees
- moved R4 149.5 mm to (248.9, 45.7), turned to 270 degrees
- moved R7 149.0 mm to (252.7, 40.6), turned to 270 degrees
- moved R2 142.9 mm to (252.7, 30.5), turned to 270 degrees
- moved R14 140.7 mm to (241.3, 45.7), turned to 270 degrees
- moved R9 140.0 mm to (245.1, 45.7), turned to 270 degrees
- moved R5 119.7 mm to (274.3, 30.5), turned to 270 degrees
- moved R12 114.9 mm to (252.7, 50.8), turned to 270 degrees
- moved R11 114.6 mm to (237.5, 50.8), turned to 270 degrees
- moved R10 111.9 mm to (270.5, 38.1), turned to 270 degrees
- moved R3 100.7 mm to (265.4, 30.5), turned to 270 degrees
- moved Q1 98.0 mm to (259.1, 30.5), turned to 270 degrees
- moved Q3 94.8 mm to (259.1, 50.8), turned to 270 degrees
- moved J1 91.5 mm to (245.1, 31.8)
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Connections:
- U2 pad 1: Net-(R1-Pad1) -> +5v
- U2 pad 10: Net-(U2-Pad10) -> Net-(R9-Pad2)
- U2 pad 11: +5v -> Net-(R6-Pad1)
- U2 pad 12: Net-(U2-Pad12) -> Net-(R4-Pad2)
- U2 pad 13: +5v -> Net-(R1-Pad1)
- U2 pad 2: Net-(R4-Pad2) -> Net-(U2-Pad2)
- U2 pad 3: Net-(R6-Pad1) -> +5v
- U2 pad 4: Net-(R9-Pad2) -> Net-(U2-Pad4)
- U2 pad 5: Net-(R11-Pad1) -> +5v
- U2 pad 6: Net-(R14-Pad2) -> Net-(U2-Pad6)
- U2 pad 8: Net-(U2-Pad8) -> Net-(R14-Pad2)
- U2 pad 9: +5v -> Net-(R11-Pad1)
Routing:
- net +5v: track 339.0 -> 498.9 mm, vias 4 -> 5
- net GND: track 520.4 -> 613.1 mm, vias 7 -> 8
- net Net-(R1-Pad1): track 0.00 -> 70.8 mm, vias 0 -> 1
- net Net-(R6-Pad1): track 0.00 -> 57.0 mm, vias 0 -> 2
- net Net-(J1-Pad2): track 0.00 -> 56.6 mm, vias 0 -> 1
- net Net-(J1-Pad1): track 0.00 -> 51.9 mm, vias 0 -> 3
- net Net-(R11-Pad1): track 0.00 -> 50.9 mm, vias 0 -> 2
- net Net-(J1-Pad3): track 0.00 -> 33.9 mm
- net Net-(J1-Pad5): track 0.00 -> 30.1 mm
- net Net-(J1-Pad4): track 0.00 -> 27.0 mm
- net Net-(R4-Pad2): track 0.00 -> 25.8 mm
- net Net-(Q1-Pad2): track 0.00 -> 23.7 mm
- net Net-(Q2-Pad2): track 0.00 -> 21.7 mm, vias 0 -> 1
- net Net-(Q3-Pad2): track 0.00 -> 20.4 mm
- net Net-(R9-Pad2): track 0.00 -> 18.4 mm
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
Commit message: expansion board
Parts:
- added Logo1: Pinnated, Pinnated:Pinnule, F.Cu at (266.7, 111.8)
- moved R1 4.02 mm to (241.3, 31.8), turned to 180 degrees
- moved R3 3.59 mm to (262.9, 33.0), turned to 0 degrees
- moved R6 1.27 mm to (237.5, 39.4)
- moved R8 1.27 mm to (265.4, 39.4)
- moved R11 1.27 mm to (237.5, 49.5)
- moved R13 1.27 mm to (265.4, 49.5)
- moved Q1 1.27 mm to (257.8, 30.5)
Routing:
- net +5v: track 498.9 -> 504.4 mm
- net Net-(R17-Pad1): track 64.3 -> 68.1 mm
- net Net-(Q1-Pad3): track 7.40 -> 5.08 mm
- net GND: track 613.1 -> 615.2 mm
- net Net-(J1-Pad3): track 33.9 -> 31.8 mm
- net Net-(R6-Pad1): track 57.0 -> 59.0 mm
- net Net-(R1-Pad1): track 70.8 -> 69.0 mm
- net Net-(R4-Pad2): track 25.8 -> 24.3 mm
- net Net-(Q1-Pad2): track 23.7 -> 22.4 mm
- net Net-(Q2-Pad3): track 7.40 -> 7.93 mm
- net Net-(Q3-Pad3): track 7.40 -> 7.93 mm
- net Net-(R11-Pad1): track 50.9 -> 50.4 mm
Other:
- board text added: "Copyright (c) 2021 andrew@pinnated.com"
- board text added: "TeleText Prototype 1 22 May 2021"

Commit message: finished and Gerbers generated
Parts:
- J2: footprint Connector_PinHeader_2.54mm:PinHeader_2x25_P2.54mm_Vertical -> Connector_IDC:IDC-Header_2x25_P2.54mm_Vertical
- Q1, Q2, Q3: footprint Package_TO_SOT_THT:TO-92_Inline -> Package_TO_SOT_THT:TO-92_Inline_Wide
- U1, U2, U3, U7: footprint Package_DIP:DIP-14_W7.62mm_LongPads -> Package_DIP:DIP-14_W7.62mm_Socket_LongPads
- U10, U8, U9: footprint Package_DIP:DIP-16_W7.62mm_LongPads -> Package_DIP:DIP-16_W7.62mm_Socket_LongPads
- U4: footprint Package_DIP:DIP-24_W15.24mm_LongPads -> Package_DIP:DIP-24_W15.24mm_Socket_LongPads
- U5: footprint Package_DIP:DIP-28_W15.24mm_LongPads -> Package_DIP:DIP-28_W15.24mm_Socket_LongPads
- U6: footprint Package_DIP:DIP-48_W15.24mm_LongPads -> Package_DIP:DIP-48_W15.24mm_Socket_LongPads
- moved C9 1.91 mm to (185.4, 101.0)
- moved Q3 1.90 mm to (259.1, 48.9)
- moved Q1 1.27 mm to (259.1, 30.5)
- moved Q2 0.63 mm to (259.1, 40.0)
- moved R3 0.63 mm to (263.5, 33.0)
Routing:
- net Net-(Q1-Pad2): track 22.4 -> 25.5 mm
- net Net-(R1-Pad1): track 69.0 -> 66.7 mm
- net Net-(J1-Pad4): track 27.0 -> 28.3 mm
- net Net-(Q3-Pad3): track 7.93 -> 9.09 mm
- net /A9: track 68.5 -> 67.3 mm
- net /A8: track 63.4 -> 62.3 mm
- net Net-(Q2-Pad3): track 7.93 -> 8.72 mm
- net Net-(J1-Pad5): track 30.1 -> 29.5 mm
- net GND: track 615.2 -> 614.5 mm
Other:
- board size 99.1 x 99.1 mm -> 100 x 100 mm
- board text added: "1"
- board text added: "Teletext Prototype 1 22 May 2021"
- board text removed: "TeleText Prototype 1 22 May 2021"
