File: hardware/6809expansion/6809expansion.sch (KiCad schematic (older format))
At the start: 13 parts, among them J0 SS50-LIKE, J1 SS50-LIKE, J2 SS50-LIKE, J3 SS50-LIKE, J4 SS50-LIKE, J5 SS50-LIKE, J6 SS50-LIKE, J7 SS50-LIKE

Commit message: finished and Gerbers generated
Parts:
- J0, J1, J2, J3, J4, J5, J6, J7: footprint Connector_PinHeader_2.54mm:PinHeader_2x25_P2.54mm_Vertical -> Connector_IDC:IDC-Header_2x25_P2.54mm_Vertical
Changed lines of the file:
@@
 F 0 "J0" H 1650 3854 45  0000 C CNN
 F 1 "SS50-LIKE" H 1650 3770 45  0000 C CNN
-F 2 "Connector_PinHeader_2.54mm:PinHeader_2x25_P2.54mm_Vertical" H 1680 2350 20  0001 C CNN
+F 2 "Connector_IDC:IDC-Header_2x25_P2.54mm_Vertical" H 1680 2350 20  0001 C CNN
 F 3 "" H 1650 2200 50  0001 C CNN
 	1    1650 2200
@@
 F 0 "J1" H 3750 3854 45  0000 C CNN
 F 1 "SS50-LIKE" H 3750 3770 45  0000 C CNN
-F 2 "Connector_PinHeader_2.54mm:PinHeader_2x25_P2.54mm_Vertical" H 3780 2350 20  0001 C CNN
+F 2 "Connector_IDC:IDC-Header_2x25_P2.54mm_Vertical" H 3780 2350 20  0001 C CNN
 F 3 "" H 3750 2200 50  0001 C CNN
 	1    3750 2200
@@
 F 0 "J2" H 5850 3854 45  0000 C CNN
 F 1 "SS50-LIKE" H 5850 3770 45  0000 C CNN
-F 2 "Connector_PinHeader_2.54mm:PinHeader_2x25_P2.54mm_Vertical" H 5880 2350 20  0001 C CNN
+F 2 "Connector_IDC:IDC-Header_2x25_P2.54mm_Vertical" H 5880 2350 20  0001 C CNN
 F 3 "" H 5850 2200 50  0001 C CNN
 	1    5850 2200
@@
 F 0 "J3" H 7950 3854 45  0000 C CNN
 F 1 "SS50-LIKE" H 7950 3770 45  0000 C CNN
-F 2 "Connector_PinHeader_2.54mm:PinHeader_2x25_P2.54mm_Vertical" H 7980 2350 20  0001 C CNN
+F 2 "Connector_IDC:IDC-Header_2x25_P2.54mm_Vertical" H 7980 2350 20  0001 C CNN
 F 3 "" H 7950 2200 50  0001 C CNN
 	1    7950 2200
@@
 F 0 "J4" H 10050 3854 45  0000 C CNN
 F 1 "SS50-LIKE" H 10050 3770 45  0000 C CNN
-F 2 "Connector_PinHeader_2.54mm:PinHeader_2x25_P2.54mm_Vertical" H 10080 2350 20  0001 C CNN
+F 2 "Connector_IDC:IDC-Header_2x25_P2.54mm_Vertical" H 10080 2350 20  0001 C CNN
 F 3 "" H 10050 2200 50  0001 C CNN
 	1    10050 2200
@@
 F 0 "J5" H 1650 7354 45  0000 C CNN
 F 1 "SS50-LIKE" H 1650 7270 45  0000 C CNN
-F 2 "Connector_PinHeader_2.54mm:PinHeader_2x25_P2.54mm_Vertical" H 1680 5850 20  0001 C CNN
+F 2 "Connector_IDC:IDC-Header_2x25_P2.54mm_Vertical" H 1680 5850 20  0001 C CNN
 F 3 "" H 1650 5700 50  0001 C CNN
 	1    1650 5700
@@
 F 0 "J6" H 3750 7354 45  0000 C CNN
 F 1 "SS50-LIKE" H 3750 7270 45  0000 C CNN
-F 2 "Connector_PinHeader_2.54mm:PinHeader_2x25_P2.54mm_Vertical" H 3780 5850 20  0001 C CNN
+F 2 "Connector_IDC:IDC-Header_2x25_P2.54mm_Vertical" H 3780 5850 20  0001 C CNN
 F 3 "" H 3750 5700 50  0001 C CNN
 	1    3750 5700
@@
 F 0 "J7" H 5850 7354 45  0000 C CNN
 F 1 "SS50-LIKE" H 5850 7270 45  0000 C CNN
-F 2 "Connector_PinHeader_2.54mm:PinHeader_2x25_P2.54mm_Vertical" H 5880 5850 20  0001 C CNN
+F 2 "Connector_IDC:IDC-Header_2x25_P2.54mm_Vertical" H 5880 5850 20  0001 C CNN
 F 3 "" H 5850 5700 50  0001 C CNN
 	1    5850 5700
